File: thermocouple_PCB/Beehive_Monitor_main_PCB/Beehive_Monitor_main_PCB.kicad_pcb (KiCad board)
At the start: 4 copper layers, 300 x 150.1 mm, 388 parts, among them IC1 LT6700HVCS6-3#PBF, IC10 AD8226ARZ, IC11 TMUX1204DGSR, IC2 AD8226ARZ, IC3 TPS54620RHLR, IC4 AD8031ARTZ-R2, IC5 TPS54620RHLR, IC6 MAX44246ASA+, IC7 MAX44246ASA+, IC8 ADA4077-4ARZ, IC9 SN74LV123ADRG4, J1 Conn_02x08_Odd_Even, J2 Conn_02x10_Odd_Even, J3 Conn_02x15_Odd_Even, J4 Conn_02x17_Odd_Even, J5 Micro_SD_Card_Det_Hirose_DM3AT, K2 HFD3_12-L2_257_, Q1 Q_NPN_BCE, Q2 Q_NPN_BCE, Q3 Q_NPN_BCE, Q4 Q_NPN_BCE, Q5 Q_NPN_BCE, Q6 Q_NPN_BCE, Q7 Q_NPN_BCE, Q8 PNP, Q9 FDS6681Z, U1 Opamp_Quad, U2 TLV3201/2, U3 Opamp_Quad, U4 Opamp_Quad, U5 TLV3201/2, U6 Opamp_Quad, U7 Opamp_Quad, U8 Opamp_Quad

Commit message: latest pcb files
Parts:
- added 3.3_V_PWR: Conn_01x02_Pin, Connector_Molex:Molex_KK-254_AE-6410-02A_1x02_P2.54mm_Vertical, F.Cu at (111.0, 193.7)
- moved PE_15 12.4 mm to (221.9, 87.2)
- moved PE_9 12.4 mm to (221.9, 120.2)
- moved PF_14 12.4 mm to (221.9, 115.1)
- moved PE_10 12.4 mm to (221.9, 94.8)
- moved PF_15 12.4 mm to (221.9, 110.0)
- moved PI_PWR 4.12 mm to (118.3, 59.8)
- moved 5_V_PWR 2.49 mm to (128.6, 59.8)
- moved R149 1.22 mm to (173.5, 161.0), turned to 90 degrees
- moved JP3 0.76 mm to (182.7, 108.4)
- moved JP5 0.47 mm to (183.2, 149.6)
- renumbered 12_V_PWR2 to 12_V_PWR_IN, 5_V_PWR1 to 5_V_PWR, Accelerometer1 to ACC, F1 to FUSE_7_A, LCD_BTNs1 to LCD_BTNs, LED_S1 to LED_S, mic_1_LDR1 to Mic_1_LDR, mic_2 to Mic_R, PI_Ribbon1 to PI_IN, PI_PWR1 to PI_PWR
Connections:
- ACC pad 2: unconnected-(Accelerometer1-Pin_2-Pad2) -> LDR_pin_1
- ACC pad 4: LDR_pin_1 -> unconnected-(Accelerometer1-Pin_4-Pad4)
- ACC pad 7: GND -> unconnected-(Accelerometer1-Pin_7-Pad7)
- ACC pad 9: unconnected-(Accelerometer1-Pin_9-Pad9) -> GND
- LCD_BTNs pad 1: LDR_pin_1 -> BTN_3
- LCD_BTNs pad 10: BTN_2 -> LDR_pin_1
- LCD_BTNs pad 11: RW -> D_5
- LCD_BTNs pad 12: RS -> EN
- LCD_BTNs pad 13: GND -> D_4
- LCD_BTNs pad 14: BTN_3 -> RS
- LCD_BTNs pad 15: EN -> RW
- LCD_BTNs pad 16: LCD_B/light -> GND
- LCD_BTNs pad 2: LDR_pin_1 -> LCD_B/light
- LCD_BTNs pad 3: D_7 -> BTN_2
- LCD_BTNs pad 4: D_6 -> LDR_pin_1
- LCD_BTNs pad 5: LDR_pin_1 -> BTN_1
- LCD_BTNs pad 7: D_5 -> D_7
- LCD_BTNs pad 8: D_4 -> LDR_pin_1
- LCD_BTNs pad 9: BTN_1 -> D_6
- PI_IN pad 10: PI_CS -> Maintainance _int
- PI_IN pad 2: Vt_bat_trig_MCU -> PI_MOSI
- PI_IN pad 4: LDR_TRIG_out_MCU -> PI_SCLK
- PI_IN pad 5: PI_MOSI -> Vt_bat_trig_MCU
- PI_IN pad 6: 6.11_kHz_out_MCU -> PI_MISO
- PI_IN pad 7: PI_SCLK -> LDR_TRIG_out_MCU
- PI_IN pad 8: Maintainance _int -> PI_CS
- PI_IN pad 9: PI_MISO -> 6.11_kHz_out_MCU
- TC_1_2 pad 10: TC_EN_2 -> LDR_pin_1
- TC_1_2 pad 11: GND -> MCU_TC_add_1
- TC_1_2 pad 12: MCU_TC_add_1 -> TC_EN_2
- TC_1_2 pad 13: TC_Sig_1 -> GND
- TC_1_2 pad 2: TC_Sig_1 -> GND
- TC_1_2 pad 3: MCU_TC_add_1 -> TC_EN_1
- TC_1_2 pad 4: GND -> MCU_TC_add_1
- TC_1_2 pad 5: TC_EN_1 -> LDR_pin_1
- TC_1_2 pad 6: unconnected-(TC_1_2-Pin_6-Pad6) -> TC_Sig_1
- TC_1_2 pad 7: LDR_pin_1 -> unconnected-(TC_1_2-Pin_7-Pad7)
- TC_1_2 pad 8: LDR_pin_1 -> unconnected-(TC_1_2-Pin_8-Pad8)
- TC_1_2 pad 9: unconnected-(TC_1_2-Pin_9-Pad9) -> TC_Sig_1
- TC_3_4 pad 10: TC_EN_4 -> LDR_pin_1
- TC_3_4 pad 11: GND -> MCU_TC_add_1
- TC_3_4 pad 12: MCU_TC_add_1 -> TC_EN_4
- TC_3_4 pad 13: TC_Sig_1 -> GND
- TC_3_4 pad 2: TC_Sig_1 -> GND
- TC_3_4 pad 3: MCU_TC_add_1 -> TC_EN_3
- TC_3_4 pad 4: GND -> MCU_TC_add_1
- TC_3_4 pad 5: TC_EN_3 -> LDR_pin_1
- TC_3_4 pad 6: unconnected-(TC_3_4-Pin_6-Pad6) -> TC_Sig_1
- TC_3_4 pad 7: LDR_pin_1 -> unconnected-(TC_3_4-Pin_7-Pad7)
- TC_3_4 pad 8: LDR_pin_1 -> unconnected-(TC_3_4-Pin_8-Pad8)
- TC_3_4 pad 9: unconnected-(TC_3_4-Pin_9-Pad9) -> TC_Sig_1
Routing:
- net 5_V: track 420.0 -> 625.8 mm, vias 2 -> 4
- net Maintainance _int: track 129.9 -> 311.5 mm, vias 0 -> 3
- net LCD_B/light: track 0.00 -> 140.7 mm
- net BTN_3: track 0.00 -> 127.6 mm
- net BTN_2: track 0.00 -> 125.7 mm
- net EN: track 0.00 -> 124.7 mm
- net BTN_1: track 0.00 -> 123.9 mm
- net RS: track 0.01 -> 120.5 mm
- net RW: track 0.00 -> 115.0 mm
- net D_4: track 0.00 -> 104.4 mm
- net MCU_TC_add_0: track 42.2 -> 142.3 mm, vias 0 -> 2
- net D_5: track 0.00 -> 99.8 mm
- net D_6: track 0.00 -> 95.4 mm
- net D_7: track 0.00 -> 91.8 mm
- net Mic_R_AA_out_to_MCU: track 58.9 -> 149.8 mm, vias 1 -> 2
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- removed copper zone on F.Cu, net Vreg_in
Other:
- board size 300 x 150.1 mm -> 257.2 x 150.1 mm
- board text added: "Beehive Monitor"
- board text added: "MAINTENANCE"
- board text added: "NUCLEO-F429ZI"
- board text added: "Plymouth"
- board text added: "University"
- board text added: "of"
- board text removed: "Maintenance"
