File: thermocouple_PCB/Beehive_Monitor_main_PCB/Beehive_Monitor_main_PCB.kicad_sch (KiCad schematic)
At the start: 388 parts, among them IC1 LT6700HVCS6-3#PBF, IC10 AD8226ARZ, IC11 TMUX1204DGSR, IC2 AD8226ARZ, IC3 TPS54620RHLR, IC4 AD8031ARTZ-R2, IC5 TPS54620RHLR, IC6 MAX44246ASA+, IC7 MAX44246ASA+, IC8 ADA4077-4ARZ, IC9 SN74LV123ADRG4, J1 Conn_02x08_Odd_Even, J2 Conn_02x10_Odd_Even, J3 Conn_02x15_Odd_Even, J4 Conn_02x17_Odd_Even, J5 Micro_SD_Card_Det_Hirose_DM3AT, K2 HFD3_12-L2_257_, Q1 Q_NPN_BCE, Q2 Q_NPN_BCE, Q3 Q_NPN_BCE, Q4 Q_NPN_BCE, Q5 Q_NPN_BCE, Q6 Q_NPN_BCE, Q7 Q_NPN_BCE, Q8 PNP, Q9 FDS6681Z, U1 Opamp_Quad, U2 TLV3201/2, U3 Opamp_Quad, U4 Opamp_Quad, U5 TLV3201/2, U6 Opamp_Quad, U7 Opamp_Quad, U8 Opamp_Quad

Commit message: latest pcb files
Parts:
- added PI_PWR2: Conn_01x02_Pin, Connector_Molex:Molex_KK-254_AE-6410-02A_1x02_P2.54mm_Vertical, symbol Connector:Conn_01x02_Pin
Connections:
- net 3.3_V_out: now also PI_PWR2.1 (Pin_1)
- net 6.11_kHz_out_MCU: now also PI_Ribbon1.9 (Pin_9); no longer PI_Ribbon1.6 (Pin_6)
- net BTN_1: now also LCD_BTNs1.5 (Pin_5); no longer LCD_BTNs1.9 (Pin_9)
- net BTN_2: now also LCD_BTNs1.3 (Pin_3); no longer LCD_BTNs1.10 (Pin_10)
- net BTN_3: now also LCD_BTNs1.1 (Pin_1); no longer LCD_BTNs1.14 (Pin_14)
- net D_4: now also LCD_BTNs1.13 (Pin_13); no longer LCD_BTNs1.8 (Pin_8)
- net D_5: now also LCD_BTNs1.11 (Pin_11); no longer LCD_BTNs1.7 (Pin_7)
- net D_6: now also LCD_BTNs1.9 (Pin_9); no longer LCD_BTNs1.4 (Pin_4)
- net D_7: now also LCD_BTNs1.7 (Pin_7); no longer LCD_BTNs1.3 (Pin_3)
- net EN: now also LCD_BTNs1.12 (Pin_12); no longer LCD_BTNs1.15 (Pin_15)
- net GND: now also Accelerometer1.9 (Pin_9), LCD_BTNs1.16 (Pin_16), TC_1_2.13 (Pin_13), TC_1_2.2 (Pin_2), TC_3_4.13 (Pin_13), TC_3_4.2 (Pin_2), PI_PWR2.2 (Pin_2); no longer Accelerometer1.7 (Pin_7), LCD_BTNs1.13 (Pin_13), TC_1_2.11 (Pin_11), TC_1_2.4 (Pin_4), TC_3_4.11 (Pin_11), TC_3_4.4 (Pin_4)
- net LCD_B/light: now also LCD_BTNs1.2 (Pin_2); no longer LCD_BTNs1.16 (Pin_16)
- net LDR_TRIG_out_MCU: now also PI_Ribbon1.7 (Pin_7); no longer PI_Ribbon1.4 (Pin_4)
- net LDR_pin_1: now also Accelerometer1.2 (Pin_2), LCD_BTNs1.10 (Pin_10), LCD_BTNs1.4 (Pin_4), LCD_BTNs1.8 (Pin_8), TC_1_2.10 (Pin_10), TC_1_2.5 (Pin_5), TC_3_4.10 (Pin_10), TC_3_4.5 (Pin_5); no longer Accelerometer1.4 (Pin_4), LCD_BTNs1.1 (Pin_1), LCD_BTNs1.2 (Pin_2), LCD_BTNs1.5 (Pin_5), TC_1_2.7 (Pin_7), TC_1_2.8 (Pin_8), TC_3_4.7 (Pin_7), TC_3_4.8 (Pin_8)
- net MCU_TC_add_1: now also TC_1_2.11 (Pin_11), TC_1_2.4 (Pin_4), TC_3_4.11 (Pin_11), TC_3_4.4 (Pin_4); no longer TC_1_2.12 (Pin_12), TC_1_2.3 (Pin_3), TC_3_4.12 (Pin_12), TC_3_4.3 (Pin_3)
- net Maintainance _int: now also PI_Ribbon1.10 (Pin_10); no longer PI_Ribbon1.8 (Pin_8)
- net PI_CS: now also PI_Ribbon1.8 (Pin_8); no longer PI_Ribbon1.10 (Pin_10)
- net PI_MISO: now also PI_Ribbon1.6 (Pin_6); no longer PI_Ribbon1.9 (Pin_9)
- net PI_MOSI: now also PI_Ribbon1.2 (Pin_2); no longer PI_Ribbon1.5 (Pin_5)
- net PI_SCLK: now also PI_Ribbon1.4 (Pin_4); no longer PI_Ribbon1.7 (Pin_7)
- net RS: now also LCD_BTNs1.14 (Pin_14); no longer LCD_BTNs1.12 (Pin_12)
- net RW: now also LCD_BTNs1.15 (Pin_15); no longer LCD_BTNs1.11 (Pin_11)
- net TC_EN_1: now also TC_1_2.3 (Pin_3); no longer TC_1_2.5 (Pin_5)
- net TC_EN_2: now also TC_1_2.12 (Pin_12); no longer TC_1_2.10 (Pin_10)
- net TC_EN_3: now also TC_3_4.3 (Pin_3); no longer TC_3_4.5 (Pin_5)
- net TC_EN_4: now also TC_3_4.12 (Pin_12); no longer TC_3_4.10 (Pin_10)
- net TC_Sig_1: now also TC_1_2.6 (Pin_6), TC_1_2.9 (Pin_9), TC_3_4.6 (Pin_6), TC_3_4.9 (Pin_9); no longer TC_1_2.13 (Pin_13), TC_1_2.2 (Pin_2), TC_3_4.13 (Pin_13), TC_3_4.2 (Pin_2)
- net Vt_bat_trig_MCU: now also PI_Ribbon1.5 (Pin_5); no longer PI_Ribbon1.2 (Pin_2)
Other:
- moved on the sheet: LED_S1
